Commit message: modifies a1 and go2

File: robots/a1_description/urdf/a1_original.urdf (robot description, URDF)
Before this commit: robot a1, 22 links, 21 joints
Links:
- added link base; visual box size=0.001 0.001 0.001
Joints:
- added joint floating_base: type fixed, parent base, child trunk, origin xyz=0 0 0 rpy=0 0 0
