Commit message: removes gazebo params and colliders for a1

File: robots/a1_description/urdf/a1.urdf (robot description, URDF)
Before this commit: robot a1, 22 links, 21 joints
Links:
- removed link FL_thigh_shoulder
- removed link FR_thigh_shoulder
- removed link RL_thigh_shoulder
- removed link RR_thigh_shoulder
- link FL_hip: geometry visual mesh filename=package://a1_description/meshes/hip.dae scale=1 1 1
- link FR_hip: geometry visual mesh filename=package://a1_description/meshes/hip.dae scale=1 1 1
- link RL_hip: geometry visual mesh filename=package://a1_description/meshes/hip.dae scale=1 1 1
- link RR_hip: geometry visual mesh filename=package://a1_description/meshes/hip.dae scale=1 1 1
- link imu_link: geometry visual box size=0.001 0.001 0.001
Joints:
- removed joint FL_hip_fixed
- removed joint FR_hip_fixed
- removed joint RL_hip_fixed
- removed joint RR_hip_fixed

Commit message: tunes a1 collider better

File: robots/a1_description/urdf/a1.urdf (robot description, URDF)
Before this commit: robot a1, 18 links, 17 joints
Links:
- link FL_thigh: geometry collision box size=0.1 0.0245 0.034; visual mesh filename=package://a1_description/meshes/thigh.dae scale=1 1 1
- link FR_thigh: geometry collision box size=0.1 0.0245 0.034; visual mesh filename=package://a1_description/meshes/thigh_mirror.dae scale=1 1 1
- link RL_thigh: geometry collision box size=0.1 0.0245 0.034; visual mesh filename=package://a1_description/meshes/thigh.dae scale=1 1 1
- link RR_thigh: geometry collision box size=0.1 0.0245 0.034; visual mesh filename=package://a1_description/meshes/thigh_mirror.dae scale=1 1 1
- link trunk: geometry collision box size=0.49 0.16 0.114; visual mesh filename=package://a1_description/meshes/trunk.dae scale=1 1 1
