Commit message: updates go1 model

File: robots/go1_description/urdf/go1_original.urdf (robot description, URDF)
Before this commit: robot go1, 45 links, 44 joints
Links:
- added link base; visual box size=0.001 0.001 0.001
- link FL_hip_rotor: geometry collision cylinder length=0.02 radius=0.035; visual cylinder length=0.02 radius=0.035
- link FL_thigh_rotor: geometry collision cylinder length=0.02 radius=0.035; visual cylinder length=0.02 radius=0.035
- link FR_hip_rotor: geometry collision cylinder length=0.02 radius=0.035; visual cylinder length=0.02 radius=0.035
- link FR_thigh_rotor: geometry collision cylinder length=0.02 radius=0.035; visual cylinder length=0.02 radius=0.035
- link RL_hip_rotor: geometry collision cylinder length=0.02 radius=0.035; visual cylinder length=0.02 radius=0.035
- link RL_thigh_rotor: geometry collision cylinder length=0.02 radius=0.035; visual cylinder length=0.02 radius=0.035
- link RR_hip_rotor: geometry collision cylinder length=0.02 radius=0.035; visual cylinder length=0.02 radius=0.035
- link RR_thigh_rotor: geometry collision cylinder length=0.02 radius=0.035; visual cylinder length=0.02 radius=0.035
- link camera_chin: mass None -> 1e-5; geometry collision box size=.001 .001 .001; visual mesh filename=package://go1_description/meshes/depthCamera.dae scale=1 1 1
- link camera_face: mass None -> 1e-5; geometry collision box size=.001 .001 .001; visual mesh filename=package://go1_description/meshes/depthCamera.dae scale=1 1 1
- link camera_left: mass None -> 1e-5; geometry collision box size=.001 .001 .001; visual mesh filename=package://go1_description/meshes/depthCamera.dae scale=1 1 1
- link camera_rearDown: mass None -> 1e-5; geometry collision box size=.001 .001 .001; visual mesh filename=package://go1_description/meshes/depthCamera.dae scale=1 1 1
- link camera_right: mass None -> 1e-5; geometry collision box size=.001 .001 .001; visual mesh filename=package://go1_description/meshes/depthCamera.dae scale=1 1 1
- link imu_link: geometry collision box size=.001 .001 .001; visual box size=0.001 0.001 0.001
- link ultraSound_face: mass None -> 1e-5; geometry collision box size=.001 .001 .001; visual mesh filename=package://go1_description/meshes/ultraSound.dae scale=1 1 1
- link ultraSound_left: mass None -> 1e-5; geometry collision box size=.001 .001 .001; visual mesh filename=package://go1_description/meshes/ultraSound.dae scale=1 1 1
- link ultraSound_right: mass None -> 1e-5; geometry collision box size=.001 .001 .001; visual mesh filename=package://go1_description/meshes/ultraSound.dae scale=1 1 1
Joints:
- added joint floating_base: type fixed, parent base, child trunk, origin xyz=0 0 0 rpy=0 0 0
