Commit message: tunes colliders to be nicer on go1

File: robots/go1_description/urdf/go1.urdf (robot description, URDF)
Before this commit: robot go1, 45 links, 44 joints
Links:
- link FL_thigh: geometry collision box size=0.1 0.0245 0.034; visual mesh filename=package://go1_description/meshes/thigh.dae scale=1 1 1
- link FR_thigh: geometry collision box size=0.1 0.0245 0.034; visual mesh filename=package://go1_description/meshes/thigh_mirror.dae scale=1 1 1
- link RL_thigh: geometry collision box size=0.1 0.0245 0.034; visual mesh filename=package://go1_description/meshes/thigh.dae scale=1 1 1
- link RR_thigh: geometry collision box size=0.1 0.0245 0.034; visual mesh filename=package://go1_description/meshes/thigh_mirror.dae scale=1 1 1
- link trunk: geometry collision box size=0.48 0.13 0.114; visual mesh filename=package://go1_description/meshes/trunk.dae scale=1 1 1
